File: kicad/pi.kicad_sch (KiCad schematic)
At the start: 10 parts, among them J2 Raspberry Pi, J3 UART console

Commit message: kicad: drop UART console and second 1-Wire terminal, tighten buck loop
Schematic: J3 (UART console) and J20 (1-Wire 2) removed by minimal
edits; Pi header pins 8/10 (GPIO14/15) marked no-connect. ERC clean,
connectivity otherwise unchanged.
Board: J3/J20 removed, S1-S4 moved up on the right edge, buck converter
placed per TI layout guidance (D4 SW pad 2.8 mm and L1 SW pad 3.7 mm
from U1-SW, input cap 3.5 mm from VIN, control parts away from SW;
>= 25.9 mm to the pH input). DRC with schematic parity: only the known
J2/Zero-hole overlap, silkscreen and unrouted nets.
Docs: 1 AKL 101-03 less, 35 header pins, cost ~40 EUR/board at 5.

Co-Authored-By: Claude Opus 5.5 <noreply@anthropic.com>
Parts:
- removed J3: UART console, Connector_PinHeader_2.54mm:PinHeader_1x03_P2.54mm_Vertical, symbol Connector_Generic:Conn_01x03
Connections:
- net GPIO14_TXD: no longer names the net of J2.8 (Pin_8)
- net GPIO15_RXD: no longer names the net of J2.10 (Pin_10)
- no-connect marks 4 -> 6
