File: kicad/aquaPCB.kicad_sch (KiCad schematic)
At the start: 0 parts

Commit message: kicad: galvanically isolate the analog / pH section
The tank water is tied to board GND through other sensors (DS18B20
sleeve), so the biased pH reference electrode would carry a continuous
DC current. Move ADS1115, pH buffer, TL431 and the AIN2/AIN3 terminals
to an isolated domain: B0505S 1 W DC/DC + AMS1117 for ISO_3V3, ISO1540
I2C isolator (side 2 on the Pi bus, side 1 on the ADS1115). Netlist
checked: only the DC/DC and the ISO1540 cross the boundary. BOM, README
and cost estimate (~45 EUR/board at 5) updated.

Co-Authored-By: Claude Opus 5.5 <noreply@anthropic.com>
Other:
- removed sheet ADS1115 ADC and pH front end
- added sheet Isolated ADC and pH front end (analog.kicad_sch)
Changed lines of the file:
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@@
+	)
+	(sheet
+		(at 182.88 38.1)
+		(size 55.88 17.78)
+		(exclude_from_sim no)
+		(in_bom yes)
+		(on_board yes)
+		(dnp no)
+		(fields_autoplaced yes)
+		(stroke
+			(width 0.1524)
+			(type solid)
+		)
+		(fill
+			(color 0 0 0 0)
+		)
+		(property "Sheetname" "Power outputs Q1..Q6"
+			(at 182.88 37.3884 0)
+			(show_name no)
+			(do_not_autoplace no)
+			(effects
+				(font
+					(size 1.27 1.27)
+				)
+				(justify left bottom)
+			)
+		)
+		(property "Sheetfile" "outputs.kicad_sch"
+			(at 182.88 56.4684 0)
+			(show_name no)
+			(do_not_autoplace no)
+			(effects
+				(font
+					(size 1.27 1.27)
+				)
+				(justify left top)
+			)
+		)
+		(instances
+			(project "aquaPCB"
+				(path "/58e047c8-5e2c-481f-8c56-e7d5c450ddf1"
+					(page "4")
+				)
+			)
+		)
+	)
+	(sheet
+		(at 106.68 76.2)
+		(size 55.88 17.78)
+		(exclude_from_sim no)
+		(in_bom yes)
+		(on_board yes)
+		(dnp no)
+		(fields_autoplaced yes)
+		(stroke
+			(width 0.1524)
+			(type solid)
+		)
+		(fill
+			(color 0 0 0 0)
+		)
+		(property "Sheetname" "Inputs, 1-Wire, I2C and display headers"
+			(at 106.68 75.4884 0)
+			(show_name no)
+			(do_not_autoplace no)
+			(effects
+				(font
+					(size 1.27 1.27)
+				)
+				(justify left bottom)
+			)
+		)
+		(property "Sheetfile" "io.kicad_sch"
+			(at 106.68 94.5684 0)
+			(show_name no)
+			(do_not_autoplace no)
+			(effects
+				(font
+					(size 1.27 1.27)
+				)
+				(justify left top)
+			)
+		)
+		(instances
+			(project "aquaPCB"
+				(path "/58e047c8-5e2c-481f-8c56-e7d5c450ddf1"
+					(page "6")
+				)
+			)
+		)
+	)
+	(sheet
+		(at 182.88 76.2)
+		(size 55.88 17.78)
+		(exclude_from_sim no)
+		(in_bom yes)
+		(on_board yes)
+		(dnp no)
+		(fields_autoplaced yes)
+		(stroke
+			(width 0.1524)
+			(type solid)
+		)
+		(fill
+			(color 0 0 0 0)
+		)
+		(property "Sheetname" "Isolated ADC and pH front end"
+			(at 182.88 75.4884 0)
+			(show_name no)
+			(do_not_autoplace no)
+			(effects
+				(font
+					(size 1.27 1.27)
+				)
+				(justify left bottom)
+			)
+		)
+		(property "Sheetfile" "analog.kicad_sch"
+			(at 182.88 94.5684 0)
+			(show_name no)
+			(do_not_autoplace no)
+			(effects
+				(font
+					(size 1.27 1.27)
+				)
+				(justify left top)
+			)
+		)
+		(instances
+			(project "aquaPCB"
+				(path "/58e047c8-5e2c-481f-8c56-e7d5c450ddf1"
+					(page "7")
+				)
+			)
+		)
 	)
 	(sheet
@@
 		(instances
 			(project "aquaPCB"
-				(path "/9dc36d06-9fe9-4bd1-aa74-847cb6598aa7"
+				(path "/58e047c8-5e2c-481f-8c56-e7d5c450ddf1"
 					(page "2")
-				)
-			)
-		)
-	)
-	(sheet
-		(at 182.88 38.1)
-		(size 55.88 17.78)
-		(exclude_from_sim no)
-		(in_bom yes)
-		(on_board yes)
-		(dnp no)
-		(fields_autoplaced yes)
-		(stroke
-			(width 0.1524)
-			(type solid)
-		)
-		(fill
-			(color 0 0 0 0)
-		)
-		(property "Sheetname" "Power outputs Q1..Q6"
-			(at 182.88 37.3884 0)
-			(show_name no)
-			(do_not_autoplace no)
-			(effects
-				(font
-					(size 1.27 1.27)
-				)
-				(justify left bottom)
-			)
-		)
-		(property "Sheetfile" "outputs.kicad_sch"
-			(at 182.88 56.4684 0)
-			(show_name no)
-			(do_not_autoplace no)
-			(effects
-				(font
-					(size 1.27 1.27)
-				)
-				(justify left top)
-			)
-		)
-		(instances
-			(project "aquaPCB"
-				(path "/9dc36d06-9fe9-4bd1-aa74-847cb6598aa7"
-					(page "4")
 				)
 			)
@@
 		(instances
 			(project "aquaPCB"
-				(path "/9dc36d06-9fe9-4bd1-aa74-847cb6598aa7"
+				(path "/58e047c8-5e2c-481f-8c56-e7d5c450ddf1"
 					(page "3")
-				)
-			)
-		)
-	)
-	(sheet
-		(at 106.68 76.2)
-		(size 55.88 17.78)
-		(exclude_from_sim no)
-		(in_bom yes)
-		(on_board yes)
-		(dnp no)
-		(fields_autoplaced yes)
-		(stroke
-			(width 0.1524)
-			(type solid)
-		)
-		(fill
-			(color 0 0 0 0)
-		)
-		(property "Sheetname" "Inputs, 1-Wire, I2C and display headers"
-			(at 106.68 75.4884 0)
-			(show_name no)
-			(do_not_autoplace no)
-			(effects
-				(font
-					(size 1.27 1.27)
-				)
-				(justify left bottom)
-			)
-		)
-		(property "Sheetfile" "io.kicad_sch"
-			(at 106.68 94.5684 0)
-			(show_name no)
-			(do_not_autoplace no)
-			(effects
-				(font
-					(size 1.27 1.27)
-				)
-				(justify left top)
-			)
-		)
-		(instances
-			(project "aquaPCB"
-				(path "/9dc36d06-9fe9-4bd1-aa74-847cb6598aa7"
-					(page "6")
-				)
-			)
-		)
-	)
-	(sheet
-		(at 182.88 76.2)
-		(size 55.88 17.78)
-		(exclude_from_sim no)
-		(in_bom yes)
-		(on_board yes)
-		(dnp no)
-		(fields_autoplaced yes)
-		(stroke
-			(width 0.1524)
-			(type solid)
-		)
-		(fill
-			(color 0 0 0 0)
-		)
-		(property "Sheetname" "ADS1115 ADC and pH front end"
-			(at 182.88 75.4884 0)
-			(show_name no)
-			(do_not_autoplace no)
-			(effects
-				(font
-					(size 1.27 1.27)
-				)
-				(justify left bottom)
-			)
-		)
-		(property "Sheetfile" "analog.kicad_sch"
-			(at 182.88 94.5684 0)
-			(show_name no)
-			(do_not_autoplace no)
-			(effects
-				(font
-					(size 1.27 1.27)
-				)
-				(justify left top)
-			)
-		)
-		(instances
-			(project "aquaPCB"
-				(path "/9dc36d06-9fe9-4bd1-aa74-847cb6598aa7"
-					(page "7")
 				)
 			)
@@
 		(instances
 			(project "aquaPCB"
-				(path "/9dc36d06-9fe9-4bd1-aa74-847cb6598aa7"
+				(path "/58e047c8-5e2c-481f-8c56-e7d5c450ddf1"
 					(page "5")
 				)

Commit message: kicad: simpler non-isolated pH amplifier after review of the hand-built setup
Nothing in the tank is grounded and ~0.1 pH stability is enough, so the
galvanic isolation (B0505S + ISO1540) and the TL431 reference go. The
on-board pH amplifier now mirrors the proven PH-4502C mod: 10 MOhm +
6.8 nF styroflex input filter, TLV9062 buffer, bias 3V3/2 buffered,
plus 1 MOhm in the reference line as ground-loop insurance. AIN2 is a
module input for 5 V amplifier boards with a 10k/20k divider (0..5 V).
BOM, README and cost (~41 EUR/board at 5, ~33 at 10) updated.

Co-Authored-By: Claude Opus 5.5 <noreply@anthropic.com>
Other:
- removed sheet Isolated ADC and pH front end
- added sheet ADS1115 ADC and pH amplifier (analog.kicad_sch)
Changed lines of the file:
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@@
 		(instances
 			(project "aquaPCB"
-				(path "/58e047c8-5e2c-481f-8c56-e7d5c450ddf1"
+				(path "/80232f81-1179-4777-a7f0-674a974d53cc"
 					(page "4")
 				)
@@
 		(instances
 			(project "aquaPCB"
-				(path "/58e047c8-5e2c-481f-8c56-e7d5c450ddf1"
+				(path "/80232f81-1179-4777-a7f0-674a974d53cc"
 					(page "6")
 				)
@@
 			(color 0 0 0 0)
 		)
-		(property "Sheetname" "Isolated ADC and pH front end"
+		(property "Sheetname" "ADS1115 ADC and pH amplifier"
 			(at 182.88 75.4884 0)
 			(show_name no)
@@
 		(instances
 			(project "aquaPCB"
-				(path "/58e047c8-5e2c-481f-8c56-e7d5c450ddf1"
+				(path "/80232f81-1179-4777-a7f0-674a974d53cc"
 					(page "7")
 				)
@@
 		(instances
 			(project "aquaPCB"
-				(path "/58e047c8-5e2c-481f-8c56-e7d5c450ddf1"
+				(path "/80232f81-1179-4777-a7f0-674a974d53cc"
 					(page "2")
+				)
+			)
+		)
+	)
+	(sheet
+		(at 30.48 76.2)
+		(size 55.88 17.78)
+		(exclude_from_sim no)
+		(in_bom yes)
+		(on_board yes)
+		(dnp no)
+		(fields_autoplaced yes)
+		(stroke
+			(width 0.1524)
+			(type solid)
+		)
+		(fill
+			(color 0 0 0 0)
+		)
+		(property "Sheetname" "SSR / relay control outputs S1..S4"
+			(at 30.48 75.4884 0)
+			(show_name no)
+			(do_not_autoplace no)
+			(effects
+				(font
+					(size 1.27 1.27)
+				)
+				(justify left bottom)
+			)
+		)
+		(property "Sheetfile" "ssr.kicad_sch"
+			(at 30.48 94.5684 0)
+			(show_name no)
+			(do_not_autoplace no)
+			(effects
+				(font
+					(size 1.27 1.27)
+				)
+				(justify left top)
+			)
+		)
+		(instances
+			(project "aquaPCB"
+				(path "/80232f81-1179-4777-a7f0-674a974d53cc"
+					(page "5")
 				)
 			)
@@
 		(instances
 			(project "aquaPCB"
-				(path "/58e047c8-5e2c-481f-8c56-e7d5c450ddf1"
+				(path "/80232f81-1179-4777-a7f0-674a974d53cc"
 					(page "3")
 				)
 			)
-		)
-	)
-	(sheet
-		(at 30.48 76.2)
-		(size 55.88 17.78)
-		(exclude_from_sim no)
-		(in_bom yes)
-		(on_board yes)
-		(dnp no)
-		(fields_autoplaced yes)
-		(stroke
-			(width 0.1524)
-			(type solid)
-		)
-		(fill
-			(color 0 0 0 0)
-		)
-		(property "Sheetname" "SSR / relay control outputs S1..S4"
-			(at 30.48 75.4884 0)
-			(show_name no)
-			(do_not_autoplace no)
-			(effects
-				(font
-					(size 1.27 1.27)
-				)
-				(justify left bottom)
-			)
-		)
-		(property "Sheetfile" "ssr.kicad_sch"
-			(at 30.48 94.5684 0)
-			(show_name no)
-			(do_not_autoplace no)
-			(effects
-				(font
-					(size 1.27 1.27)
-				)
-				(justify left top)
-			)
-		)
-		(instances
-			(project "aquaPCB"
-				(path "/58e047c8-5e2c-481f-8c56-e7d5c450ddf1"
-					(page "5")
-				)
-			)

Commit message: kicad: routing progress (by hand)
Co-Authored-By: Claude Opus 5.5 (1M context) <noreply@anthropic.com>
Changed lines of the file:
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@@
 	(generator "eeschema")
 	(generator_version "10.0")
-	(paper "A4")
+	(paper "A4" portrait)
 	(title_block
 		(title "aquaPCB – Overview")
@@
 	)
 	(sheet
-		(at 182.88 38.1)
+		(at 30.48 76.2)
 		(size 55.88 17.78)
 		(exclude_from_sim no)
@@
 		)
 		(property "Sheetname" "Power outputs Q1..Q6"
-			(at 182.88 37.3884 0)
+			(at 30.48 75.4884 0)
 			(show_name no)
 			(do_not_autoplace no)
@@
 		)
 		(property "Sheetfile" "outputs.kicad_sch"
-			(at 182.88 56.4684 0)
+			(at 30.48 94.5684 0)
 			(show_name no)
 			(do_not_autoplace no)
@@
 	)
 	(sheet
-		(at 106.68 76.2)
+		(at 30.48 113.03)
 		(size 55.88 17.78)
 		(exclude_from_sim no)
@@
 		)
 		(property "Sheetname" "Inputs, 1-Wire, I2C and display headers"
-			(at 106.68 75.4884 0)
+			(at 30.48 112.3184 0)
 			(show_name no)
 			(do_not_autoplace no)
@@
 		)
 		(property "Sheetfile" "io.kicad_sch"
-			(at 106.68 94.5684 0)
+			(at 30.48 131.3984 0)
 			(show_name no)
 			(do_not_autoplace no)
@@
 	)
 	(sheet
-		(at 182.88 76.2)
+		(at 106.68 113.03)
 		(size 55.88 17.78)
 		(exclude_from_sim no)
@@
 		)
 		(property "Sheetname" "ADS1115 ADC and pH amplifier"
-			(at 182.88 75.4884 0)
+			(at 106.68 112.3184 0)
 			(show_name no)
 			(do_not_autoplace no)
@@
 		)
 		(property "Sheetfile" "analog.kicad_sch"
-			(at 182.88 94.5684 0)
+			(at 106.68 131.3984 0)
 			(show_name no)
 			(do_not_autoplace no)
@@
 	)
 	(sheet
-		(at 30.48 76.2)
+		(at 106.68 76.2)
 		(size 55.88 17.78)
 		(exclude_from_sim no)
@@
 		)
 		(property "Sheetname" "SSR / relay control outputs S1..S4"
-			(at 30.48 75.4884 0)
+			(at 106.68 75.4884 0)
 			(show_name no)
 			(do_not_autoplace no)
@@
 		)
 		(property "Sheetfile" "ssr.kicad_sch"
-			(at 30.48 94.5684 0)
-			(show_name no)
-			(do_not_autoplace no)
+			(at 106.68 94.5684 0)
+			(show_name no)
+			(do_not_autoplace no)
