File: kicad/ssr.kicad_sch (KiCad schematic)
At the start: 14 parts, among them J11 GPIO 17, J12 GPIO 22, J13 GPIO 23, J14 GPIO 27, U4 ULN2803A

Commit message: kicad: schematic re-save (library symbol refresh, BOM field setup)
Parts:
- D18, D19, D20, D21, R32, R33, R34, R35: KiLib_Generator (none) -> SMD_2terminal_chip_molded
- J11, J12, J13, J14: KiLib_Generator (none) -> terminal_block/Phoenix
- JP2: KiLib_Generator (none) -> connector/pin_header_socket
- U4: KiLib_Generator (none) -> package/gullwing
