File: kicad/aquaPCB.kicad_pcb (KiCad board)
At the start: 2 copper layers, 100 x 100 mm, 149 parts, among them J1 12V IN, J11 SSR G17, J12 SSR G22, J13 SSR G23, J14 SSR G27, J15 IN1, J16 IN2, J17 IN3, J18 IN4, J19 1-Wire 1, J2 Raspberry Pi, J22 I2C 1, J23 I2C 2, J24 Display, J25 pH probe, J26 Module, J27 AIN3, J4 OUT G18, J5 OUT G19, J6 OUT G12, J7 OUT G13, J8 OUT G16, J9 OUT G26, Q1 AOD4184A, Q10 AOD4185, Q2 AOD4184A, Q3 AOD4184A, Q4 AOD4184A, Q5 AOD4184A, Q6 AOD4184A, U1 TPS54360B, U2 AMS1117-3.3, U3 74HCT244D, U4 ULN2803A, U5 ADS1115IDGSR, U6 TLV9062IDR

Commit message: kicad: reorder 74HCT244 channels for crossing-free Pi -> driver routing
Inputs enter U3 from outside (pull-downs R8..R13 as a staircase), outputs
leave inside under the IC body towards Q1..Q6. The GPIO order on the Pi
header then has to be Q6..Q1, so the stage mapping changes to
Q2 = GPIO12, Q3 = GPIO13, Q4 = GPIO19 (hardware PWM stays on GPIO18/19,
now Q1/Q4). Unused channels: pin 8/11 inputs to GND, pin 9/12 open.

Co-Authored-By: Claude Opus 5.5 <noreply@anthropic.com>
Parts:
- D11: value GPIO12 -> GPIO13
- D13: value GPIO13 -> GPIO19
- D9: value GPIO19 -> GPIO12
Connections:
- J2 pad 32: GPIO12_Q3 -> GPIO12_Q2
- J2 pad 33: GPIO13_Q4 -> GPIO13_Q3
- J2 pad 35: GPIO19_Q2 -> GPIO19_Q4
- R10 pad 1: GPIO12_Q3 -> GPIO26_Q6
- R11 pad 1: GPIO13_Q4 -> GPIO13_Q3
- R12 pad 1: GPIO16_Q5 -> GPIO12_Q2
- R13 pad 1: GPIO26_Q6 -> GPIO18_Q1
- R8 pad 1: GPIO18_Q1 -> GPIO19_Q4
- R9 pad 1: GPIO19_Q2 -> GPIO16_Q5
- U3 pad 12: /Power outputs Q1..Q6/Q4_DRV -> unconnected-(U3-1Y3-Pad12)
- U3 pad 13: GND -> GPIO18_Q1
- U3 pad 14: /Power outputs Q1..Q6/Q3_DRV -> /Power outputs Q1..Q6/Q6_DRV
- U3 pad 15: GPIO26_Q6 -> GPIO12_Q2
- U3 pad 16: /Power outputs Q1..Q6/Q2_DRV -> /Power outputs Q1..Q6/Q5_DRV
- U3 pad 17: GPIO16_Q5 -> GPIO13_Q3
- U3 pad 18: /Power outputs Q1..Q6/Q1_DRV -> /Power outputs Q1..Q6/Q4_DRV
- U3 pad 2: GPIO18_Q1 -> GPIO19_Q4
- U3 pad 3: /Power outputs Q1..Q6/Q5_DRV -> /Power outputs Q1..Q6/Q3_DRV
- U3 pad 4: GPIO19_Q2 -> GPIO16_Q5
- U3 pad 5: /Power outputs Q1..Q6/Q6_DRV -> /Power outputs Q1..Q6/Q2_DRV
- U3 pad 6: GPIO12_Q3 -> GPIO26_Q6
- U3 pad 7: unconnected-(U3-2Y2-Pad7) -> /Power outputs Q1..Q6/Q1_DRV
- U3 pad 8: GPIO13_Q4 -> GND
Changed lines of the file:
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@@
 			)
 		)
-		(property "Value" "GPIO13"
+		(property "Value" "GPIO19"
 			(at 0 1.65 0)
 			(layer "F.Fab")
@@
 			(layers "F.Cu" "F.Mask" "F.Paste")
 			(roundrect_rratio 0.25)
-			(net "GPIO18_Q1")
+			(net "GPIO19_Q4")
 			(pinfunction "1A0_2")
 			(pintype "input")
@@
 			(layers "F.Cu" "F.Mask" "F.Paste")
 			(roundrect_rratio 0.25)
-			(net "/Power outputs Q1..Q6/Q5_DRV")
+			(net "/Power outputs Q1..Q6/Q3_DRV")
 			(pinfunction "2Y0_3")
 			(pintype "tri_state")
@@
 			(layers "F.Cu" "F.Mask" "F.Paste")
 			(roundrect_rratio 0.25)
-			(net "GPIO19_Q2")
+			(net "GPIO16_Q5")
 			(pinfunction "1A1_4")
 			(pintype "input")
@@
 			(layers "F.Cu" "F.Mask" "F.Paste")
 			(roundrect_rratio 0.25)
-			(net "/Power outputs Q1..Q6/Q6_DRV")
+			(net "/Power outputs Q1..Q6/Q2_DRV")
 			(pinfunction "2Y1_5")
 			(pintype "tri_state")
@@
 			(layers "F.Cu" "F.Mask" "F.Paste")
 			(roundrect_rratio 0.25)
-			(net "GPIO12_Q3")
+			(net "GPIO26_Q6")
 			(pinfunction "1A2_6")
 			(pintype "input")
@@
 			(layers "F.Cu" "F.Mask" "F.Paste")
 			(roundrect_rratio 0.25)
-			(net "unconnected-(U3-2Y2-Pad7)")
+			(net "/Power outputs Q1..Q6/Q1_DRV")
 			(pinfunction "2Y2_7")
 			(pintype "tri_state+no_connect")
@@
 			(layers "F.Cu" "F.Mask" "F.Paste")
 			(roundrect_rratio 0.25)
-			(net "GPIO13_Q4")
+			(net "GND")
 			(pinfunction "1A3_8")
 			(pintype "input")
@@
 			(layers "F.Cu" "F.Mask" "F.Paste")
 			(roundrect_rratio 0.25)
-			(net "/Power outputs Q1..Q6/Q4_DRV")
+			(net "unconnected-(U3-1Y3-Pad12)")
 			(pinfunction "1Y3_12")
 			(pintype "tri_state")
@@
 			(layers "F.Cu" "F.Mask" "F.Paste")
 			(roundrect_rratio 0.25)
-			(net "GND")
+			(net "GPIO18_Q1")
 			(pinfunction "2A2_13")
 			(pintype "input")
@@
 			(layers "F.Cu" "F.Mask" "F.Paste")
 			(roundrect_rratio 0.25)
-			(net "/Power outputs Q1..Q6/Q3_DRV")
+			(net "/Power outputs Q1..Q6/Q6_DRV")
 			(pinfunction "1Y2_14")
 			(pintype "tri_state")
@@
 			(layers "F.Cu" "F.Mask" "F.Paste")
 			(roundrect_rratio 0.25)
-			(net "GPIO26_Q6")
+			(net "GPIO12_Q2")
 			(pinfunction "2A1_15")
 			(pintype "input")
@@
 			(layers "F.Cu" "F.Mask" "F.Paste")
 			(roundrect_rratio 0.25)
-			(net "/Power outputs Q1..Q6/Q2_DRV")
+			(net "/Power outputs Q1..Q6/Q5_DRV")
 			(pinfunction "1Y1_16")
 			(pintype "tri_state")
@@
 			(layers "F.Cu" "F.Mask" "F.Paste")
 			(roundrect_rratio 0.25)
-			(net "GPIO16_Q5")
+			(net "GPIO13_Q3")
 			(pinfunction "2A0_17")
 			(pintype "input")
@@
 			(layers "F.Cu" "F.Mask" "F.Paste")
 			(roundrect_rratio 0.25)
-			(net "/Power outputs Q1..Q6/Q1_DRV")
+			(net "/Power outputs Q1..Q6/Q4_DRV")
 			(pinfunction "1Y0_18")
 			(pintype "tri_state")
@@
 			(layers "F.Cu" "F.Mask" "F.Paste")
 			(roundrect_rratio 0.243902)
-			(net "GPIO18_Q1")
+			(net "GPIO19_Q4")
 			(pintype "passive")
 		)
@@
 			(layers "F.Cu" "F.Mask" "F.Paste")
 			(roundrect_rratio 0.243902)
-			(net "GPIO12_Q3")
+			(net "GPIO26_Q6")
 			(pintype "passive")
 		)
@@
 			(layers "F.Cu" "F.Mask" "F.Paste")
 			(roundrect_rratio 0.243902)
-			(net "GPIO13_Q4")
+			(net "GPIO13_Q3")
 			(pintype "passive")
 		)
@@
 			(layers "*.Cu" "*.Mask")
 			(remove_unused_layers no)
-			(net "GPIO12_Q3")
+			(net "GPIO12_Q2")
 			(pinfunction "Pin_32_32")
 			(pintype "passive")
@@
 			(layers "*.Cu" "*.Mask")
 			(remove_unused_layers no)
-			(net "GPIO13_Q4")
+			(net "GPIO13_Q3")
 			(pinfunction "Pin_33_33")
 			(pintype "passive")
@@
 			(layers "*.Cu" "*.Mask")
 			(remove_unused_layers no)
-			(net "GPIO19_Q2")
+			(net "GPIO19_Q4")
 			(pinfunction "Pin_35_35")
 			(pintype "passive")
@@
 			(layers "F.Cu" "F.Mask" "F.Paste")
 			(roundrect_rratio 0.243902)
-			(net "GPIO26_Q6")
+			(net "GPIO18_Q1")
 			(pintype "passive")
 		)
@@
 			)
 		)
-		(property "Value" "GPIO19"
+		(property "Value" "GPIO12"
 			(at 0 1.65 0)
 			(layer "F.Fab")
@@
 			(layers "F.Cu" "F.Mask" "F.Paste")
 			(roundrect_rratio 0.243902)
-			(net "GPIO19_Q2")
+			(net "GPIO16_Q5")
 			(pintype "passive")
 		)
@@
 			)
 		)
-		(property "Value" "GPIO12"
+		(property "Value" "GPIO13"
 			(at 0 1.65 0)
 			(layer "F.Fab")
@@
 			(layers "F.Cu" "F.Mask" "F.Paste")
 			(roundrect_rratio 0.243902)
-			(net "GPIO16_Q5")
+			(net "GPIO12_Q2")
 			(pintype "passive")
 		)
