File: kicad/aquaPCB.kicad_pcb (KiCad board)
At the start: 2 copper layers, 100 x 100 mm, 149 parts, among them J1 12V IN, J11 SSR G17, J12 SSR G22, J13 SSR G23, J14 SSR G27, J15 IN1, J16 IN2, J17 IN3, J18 IN4, J19 1-Wire 1, J2 Raspberry Pi, J22 I2C 1, J23 I2C 2, J24 Display, J25 pH probe, J26 Module, J27 AIN3, J4 OUT G18, J5 OUT G19, J6 OUT G12, J7 OUT G13, J8 OUT G16, J9 OUT G26, Q1 AOD4184A, Q10 AOD4185, Q2 AOD4184A, Q3 AOD4184A, Q4 AOD4184A, Q5 AOD4184A, Q6 AOD4184A, U1 TPS54360B, U2 AMS1117-3.3, U3 74HCT244D, U4 ULN2803A, U5 ADS1115IDGSR, U6 TLV9062IDR

Commit message: kicad: remove dangling Q5/Q6_DRV stubs and unconnected +5V via
Co-Authored-By: Claude Opus 5.5 <noreply@anthropic.com>
Routing:
- net +5V: vias 4 -> 3
Changed lines of the file:
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@@
-	)
-	(segment
-		(start 135 103.945)
-		(end 134.945 103.945)
-		(width 0.25)
-		(layer "F.Cu")
-		(net "/Power outputs Q1..Q6/Q6_DRV")
 	)
 	(segment
@@
 		(end 111.834314 98.9)
 		(width 0.2)
-		(layer "F.Cu")
-		(net "/Power outputs Q1..Q6/Q5_DRV")
-	)
-	(segment
-		(start 135 104.395)
-		(end 134.758604 104.395)
-		(width 0.25)
 		(layer "F.Cu")
 		(net "/Power outputs Q1..Q6/Q5_DRV")
@@
 		(size 0.6)
 		(drill 0.3)
-		(layers "F.Cu" "B.Cu")
-		(net "+5V")
-	)
-	(via
-		(at 156.923008 94.923008)
-		(size 0.6)
-		(drill 0.3)
