File: kicad/aquaPCB.kicad_pcb (KiCad board)
At the start: 2 copper layers, 100 x 100 mm, 149 parts, among them J1 12V IN, J11 SSR G17, J12 SSR G22, J13 SSR G23, J14 SSR G27, J15 IN1, J16 IN2, J17 IN3, J18 IN4, J19 1-Wire 1, J2 Raspberry Pi, J22 I2C 1, J23 I2C 2, J24 Display, J25 pH probe, J26 Module, J27 AIN3, J4 OUT G18, J5 OUT G19, J6 OUT G12, J7 OUT G13, J8 OUT G16, J9 OUT G26, Q1 AOD4184A, Q10 AOD4185, Q2 AOD4184A, Q3 AOD4184A, Q4 AOD4184A, Q5 AOD4184A, Q6 AOD4184A, U1 TPS54360B, U2 AMS1117-3.3, U3 74HCT244D, U4 ULN2803A, U5 ADS1115IDGSR, U6 TLV9062IDR

Commit message: kicad: extended ground/VIN rework attempt (by hand)
Routing:
- net VIN: track 342.1 -> 365.2 mm, vias 10 -> 12
Changed lines of the file:
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@@
+	)
+	(segment
+		(start 97.785 125.5)
+		(end 97.785 126.74)
+		(width 3)
+		(layer "F.Cu")
+		(net "VIN")
 	)
 	(segment
@@
 	(segment
 		(start 97.785 122.28)
-		(end 97.785 126.74)
+		(end 97.785 125.5)
 		(width 3)
 		(layer "F.Cu")
@@
 	)
 	(via
+		(at 97.785 125.5)
+		(size 0.6)
+		(drill 0.3)
+		(layers "F.Cu" "B.Cu")
+		(net "VIN")
+	)
+	(via
 		(at 97.35 126.175)
 		(size 0.6)
@@
 	(via
 		(at 97.35 127.675)
+		(size 0.6)
+		(drill 0.3)
+		(layers "F.Cu" "B.Cu")
+		(net "VIN")
+	)
+	(via
+		(at 97.785 126.74)
 		(size 0.6)
 		(drill 0.3)
@@
 	)
 	(segment
+		(start 164.064999 105.064999)
+		(end 162.5 103.5)
+		(width 3)
+		(layer "B.Cu")
+		(net "VIN")
+	)
+	(segment
 		(start 117.075 127.93)
 		(end 117.075 123.45)
@@
 	)
 	(segment
+		(start 139.5 100)
+		(end 139.5 99.5)
+		(width 3)
+		(layer "B.Cu")
+		(net "VIN")
+	)
+	(segment
 		(start 128.425 123.6)
 		(end 128.85 123.175)
@@
 	)
 	(segment
+		(start 162.5 103.5)
+		(end 143 103.5)
+		(width 3)
+		(layer "B.Cu")
+		(net "VIN")
+	)
+	(segment
 		(start 105.725 127.8)
 		(end 110.35 123.175)
@@
 	)
 	(segment
+		(start 164.064999 119.460001)
+		(end 164.064999 105.064999)
+		(width 3)
+		(layer "B.Cu")
+		(net "VIN")
+	)
+	(segment
 		(start 135.85 123.175)
 		(end 139.85 123.175)
@@
 	)
 	(segment
+		(start 143 103.5)
+		(end 139.5 100)
+		(width 3)
+		(layer "B.Cu")
+		(net "VIN")
+	)
+	(segment
 		(start 151.125 123.4)
 		(end 151.35 123.175)
@@
 	)
 	(segment
-		(start 131.5 99.5)
-		(end 131.5 123.175)
-		(width 3)
-		(layer "B.Cu")
-		(net "VIN")
-	)
-	(segment
 		(start 105.725 127.93)
 		(end 105.725 126.904517)
@@
 		(width 3)
 		(layer "B.Cu")
+		(net "VIN")
+	)
+	(segment
+		(start 160.35 123.175)
+		(end 164.064999 119.460001)
+		(width 3)
+		(layer "B.Cu")
