File: kicad/aquaPCB.kicad_pcb (KiCad board)
At the start: 2 copper layers, 100 x 100 mm, 149 parts, among them J1 12V IN, J11 SSR G17, J12 SSR G22, J13 SSR G23, J14 SSR G27, J15 IN1, J16 IN2, J17 IN3, J18 IN4, J19 1-Wire 1, J2 Raspberry Pi, J22 I2C 1, J23 I2C 2, J24 Display, J25 pH probe, J26 Module, J27 AIN3, J4 OUT G18, J5 OUT G19, J6 OUT G12, J7 OUT G13, J8 OUT G16, J9 OUT G26, Q1 AOD4184A, Q10 AOD4185, Q2 AOD4184A, Q3 AOD4184A, Q4 AOD4184A, Q5 AOD4184A, Q6 AOD4184A, U1 TPS54360B, U2 AMS1117-3.3, U3 74HCT244D, U4 ULN2803A, U5 ADS1115IDGSR, U6 TLV9062IDR

Commit message: kicad: remove leftover stubs, no-net tracks and unconnected vias
Co-Authored-By: Claude Opus 5.5 <noreply@anthropic.com>
Routing:
- net /Power outputs Q1..Q6/Q3_DRV: track 33.7 -> 32.7 mm
- net VIN: vias 12 -> 10
- net +5V: vias 6 -> 5
Changed lines of the file:
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@@
 	)
 	(segment
-		(start 151.5 73.303299)
-		(end 151.615 73.418299)
-		(width 0.25)
-		(layer "F.Cu")
-		(net "")
-	)
-	(segment
-		(start 151.5 73)
-		(end 151.5 73.303299)
-		(width 0.25)
-		(layer "F.Cu")
-		(net "")
-	)
-	(segment
 		(start 102.605 110.5)
 		(end 104.975 112.87)
@@
 	)
 	(segment
-		(start 124.687499 105.187499)
-		(end 124.687499 106.17)
-		(width 0.25)
-		(layer "F.Cu")
-		(net "/Power outputs Q1..Q6/Q3_DRV")
-	)
-	(segment
 		(start 108.9625 103.326104)
 		(end 108.9625 93.4625)
@@
 	)
 	(via
-		(at 140 87.175)
-		(size 0.6)
-		(drill 0.3)
-		(layers "F.Cu" "B.Cu")
-		(net "VIN")
-	)
-	(via
 		(at 98.85 124.73)
 		(size 0.6)
@@
 	)
 	(via
-		(at 140 90.175)
-		(size 0.6)
-		(drill 0.3)
-		(layers "F.Cu" "B.Cu")
-		(net "VIN")
-	)
-	(via
 		(at 97.35 127.675)
 		(size 0.6)
@@
 	)
 	(segment
-		(start 107.984999 98.515001)
-		(end 108.0625 98.592501)
-		(width 0.25)
-		(layer "F.Cu")
-		(net "/Power outputs Q1..Q6/Q1_DRV")
-	)
-	(segment
 		(start 106.35 97.905)
 		(end 107.374999 97.905)
@@
 	)
 	(segment
-		(start 98.575 92.425)
-		(end 98.575 92.5)
-		(width 0.2)
-		(layer "F.Cu")
-		(net "GPIO26_Q6")
-	)
-	(segment
 		(start 98.575 92.5)
 		(end 98.575 98.649999)
@@
 	)
 	(segment
-		(start 134 103.945)
-		(end 133.945 103.945)
-		(width 0.2)
-		(layer "F.Cu")
-		(net "/Power outputs Q1..Q6/Q6_DRV")
-	)
-	(segment
 		(start 114.595 97.905)
 		(end 114 98.5)
@@
 		(size 0.6)
 		(drill 0.3)
-		(layers "F.Cu" "B.Cu")
-		(net "+5V")
-	)
-	(via
-		(at 158.5 94.825)
-		(size 0.6)
-		(drill 0.3)
