File: kicad/aquaPCB.kicad_pcb (KiCad board)
At the start: 2 copper layers, 100 x 100 mm, 149 parts, among them J1 12V IN, J11 GPIO 17, J12 GPIO 22, J13 GPIO 23, J14 GPIO 27, J15 GPIO 5, J16 GPIO 6, J17 GPIO 20, J18 GPIO 21, J19 DS1820, J2 Raspberry Pi, J22 I2C 1, J23 I2C 2, J24 Display, J25 ADC #1 in 0, J26 ADC #1 in 2, J27 ADC #1 in 3, J4 PWM 0, J5 GPIO 12, J6 GPIO 13, J7 PWM 1, J8 GPIO 16, J9 GPIO 26, Q1 AOD4184A, Q10 AOD4185, Q2 AOD4184A, Q3 AOD4184A, Q4 AOD4184A, Q5 AOD4184A, Q6 AOD4184A, U1 TPS54360B, U2 AMS1117-3.3, U3 74HCT244D, U4 ULN2803A, U5 ADS1115IDGSR, U6 TLV9062IDR

Commit message: kicad: layout tweaks (by hand)
Parts:
- D3: value PWR, red -> PWR
- D5: value 3V3, green -> 3V3
Changed lines of the file:
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@@
 			)
 		)
-		(property "Value" "PWR, red"
+		(property "Value" "PWR"
 			(at 0 1.65 0)
 			(layer "F.Fab")
@@
 			)
 		)
-		(property "Value" "3V3, green"
+		(property "Value" "3V3"
 			(at 0 1.65 90)
 			(layer "F.Fab")
