File: kicad/analog.kicad_sch (KiCad schematic)
At the start: 23 parts, among them J25 pH probe, J26 Module, J27 AIN3, U5 ADS1115IDGSR, U6 TLV9062IDR

Commit message: kicad: right-angle BNC (LCSC C49352232) at the board edge
New project footprint BNC_HanElectricity_BNC-Q9-50KWE_Horizontal, made
from the LCSC/EasyEDA pad data and the maker drawing: pad 1 = centre
contact on the axis, pad 2 = shell pin and both mounting legs; body
front face on the board edge, barrel protrudes 21.4 mm. J25 swapped on
the board with nets and schematic link kept (front face at x = 0).
ERC clean; DRC with schematic parity: no J25 findings besides unrouted
nets. Docs: BNC sourced from LCSC, shell = PH_SHELL (insulate from a
metal enclosure), insulation resistance only >= 5 GOhm; cost ~39 EUR.

Co-Authored-By: Claude Opus 5.5 <noreply@anthropic.com>
Parts:
- J25: footprint Connector_Coaxial:BNC_Amphenol_031-5539_Vertical -> aquaPCB:BNC_HanElectricity_BNC-Q9-50KWE_Horizontal; LCSC (none) -> C49352232; Reichelt UG 1094PL -> (none)
Changed lines of the file:
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@@
 			)
 		)
-		(property "Footprint" "Connector_Coaxial:BNC_Amphenol_031-5539_Vertical"
+		(property "Footprint" "aquaPCB:BNC_HanElectricity_BNC-Q9-50KWE_Horizontal"
 			(at 35.56 110.49 0)
 			(hide yes)
@@
 			)
 		)
-		(property "Reichelt" "UG 1094PL"
+		(property "LCSC" "C49352232"
 			(at 35.56 110.49 0)
 			(hide yes)

Commit message: kicad: push-in spring terminals (Kangnex WJ250B), 8 A total
All 18 screw terminals replaced by Ningbo Kangnex WJ250B push-in spring
terminals (LCSC C8454 2-pole, C8420 3-pole; 3.5 mm pitch, staggered
pins, 8 A IEC). New footprints from the EasyEDA pad data and the maker
drawing (wire entry on the pin-1 side, facing the board edge) and
simple 3D models. Board total current reduced to 8 A: fuse 8 A
(Littelfuse 0154008.DR, LCSC C206919). Board: footprints swapped with
nets and schematic links kept, edges re-placed for the deeper bodies.
ERC 0; DRC unchanged (known J2/Zero-hole overlap, silk, unrouted).
Docs: BOM/README (8 A budget, 5.3 mm input path, cost ~35 EUR/board).

Co-Authored-By: Claude Opus 5.5 <noreply@anthropic.com>
Parts:
- J26, J27: footprint TerminalBlock_Phoenix:TerminalBlock_Phoenix_MKDS-1,5-3-5.08_1x03_P5.08mm_Horizontal -> aquaPCB:TerminalBlock_Kangnex_WJ250B-3.5-03P_P3.50mm_Staggered; LCSC (none) -> C8420; Reichelt AKL 101-03 -> (none)
Changed lines of the file:
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@@
 			)
 		)
-		(property "Footprint" "TerminalBlock_Phoenix:TerminalBlock_Phoenix_MKDS-1,5-3-5.08_1x03_P5.08mm_Horizontal"
+		(property "Footprint" "aquaPCB:TerminalBlock_Kangnex_WJ250B-3.5-03P_P3.50mm_Staggered"
 			(at 35.56 246.38 0)
 			(hide yes)
@@
 			)
 		)
-		(property "Reichelt" "AKL 101-03"
+		(property "LCSC" "C8420"
 			(at 35.56 246.38 0)
 			(hide yes)
@@
 			)
 		)
-		(property "Footprint" "TerminalBlock_Phoenix:TerminalBlock_Phoenix_MKDS-1,5-3-5.08_1x03_P5.08mm_Horizontal"
+		(property "Footprint" "aquaPCB:TerminalBlock_Kangnex_WJ250B-3.5-03P_P3.50mm_Staggered"
 			(at 35.56 205.74 0)
 			(hide yes)
@@
 			)
 		)
-		(property "Reichelt" "AKL 101-03"
+		(property "LCSC" "C8420"
 			(at 35.56 205.74 0)
 			(hide yes)

Commit message: kicad: routing progress (by hand)
Co-Authored-By: Claude Opus 5.5 (1M context) <noreply@anthropic.com>
Changed lines of the file:
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@@
 	(generator "eeschema")
 	(generator_version "10.0")
-	(paper "A3")
+	(paper "A4" portrait)
 	(title_block
 		(title "aquaPCB – ADS1115 ADC and pH amplifier")
@@
 	)
 	(junction
-		(at 55.88 246.38)
-		(diameter 0)
-		(color 0 0 0 0)
-	)
-	(junction
 		(at 48.26 143.51)
 		(diameter 0)
@@
 	)
 	(junction
-		(at 64.77 205.74)
+		(at 55.88 246.38)
 		(diameter 0)
 		(color 0 0 0 0)
@@
 	)
 	(junction
+		(at 83.82 208.28)
+		(diameter 0)
+		(color 0 0 0 0)
+	)
+	(junction
+		(at 73.66 247.65)
+		(diameter 0)
+		(color 0 0 0 0)
+	)
+	(junction
 		(at 44.45 238.76)
 		(diameter 0)
@@
 	)
 	(junction
+		(at 64.77 205.74)
+		(diameter 0)
+		(color 0 0 0 0)
+	)
+	(junction
 		(at 100.33 113.03)
 		(diameter 0)
@@
 	(wire
 		(pts
+			(xy 72.39 208.28) (xy 83.82 208.28)
+		)
+		(stroke
+			(width 0)
+			(type default)
+		)
+	)
+	(wire
+		(pts
 			(xy 60.96 66.04) (xy 58.42 66.04)
 		)
@@
 	(wire
 		(pts
+			(xy 63.5 247.65) (xy 73.66 247.65)
+		)
+		(stroke
+			(width 0)
+			(type default)
+		)
+	)
+	(wire
+		(pts
 			(xy 73.66 146.05) (xy 76.2 146.05)
 		)
@@
 	(wire
 		(pts
-			(xy 55.88 246.38) (xy 55.88 245.11)
+			(xy 44.45 203.2) (xy 44.45 199.39)
 		)
 		(stroke
@@
 	(wire
 		(pts
-			(xy 44.45 203.2) (xy 44.45 199.39)
+			(xy 72.39 205.74) (xy 64.77 205.74)
 		)
 		(stroke
@@
 	(wire
 		(pts
+			(xy 83.82 208.28) (xy 86.36 208.28)
+		)
+		(stroke
+			(width 0)
+			(type default)
+		)
+	)
+	(wire
+		(pts
 			(xy 100.33 121.92) (xy 100.33 113.03)
 		)
@@
 	(wire
 		(pts
-			(xy 55.88 121.92) (xy 55.88 124.46)
+			(xy 63.5 246.38) (xy 55.88 246.38)
 		)
 		(stroke
@@
 	(wire
 		(pts
-			(xy 73.66 247.65) (xy 76.2 247.65)
+			(xy 63.5 247.65) (xy 63.5 246.38)
+		)
+		(stroke
+			(width 0)
+			(type default)
+		)
+	)
+	(wire
+		(pts
+			(xy 55.88 121.92) (xy 55.88 124.46)
 		)
 		(stroke
@@
 	(wire
 		(pts
+			(xy 72.39 208.28) (xy 72.39 205.74)
+		)
+		(stroke
+			(width 0)
+			(type default)
+		)
+	)
+	(wire
+		(pts
 			(xy 71.12 71.12) (xy 71.12 73.66)
 		)
@@
 	(wire
 		(pts
-			(xy 73.66 205.74) (xy 64.77 205.74)
-		)
-		(stroke
-			(width 0)
-			(type default)
-		)
-	)
-	(wire
-		(pts
 			(xy 55.88 132.08) (xy 55.88 124.46)
 		)
@@
 	(wire
 		(pts
-			(xy 83.82 208.28) (xy 86.36 208.28)
+			(xy 53.34 246.38) (xy 55.88 246.38)
 		)
 		(stroke
@@
 	(wire
 		(pts
-			(xy 53.34 246.38) (xy 55.88 246.38)
+			(xy 73.66 247.65) (xy 76.2 247.65)
 		)
 		(stroke
@@
 	)
 	(label "PH_REF"
+		(at 76.2 139.7 0)
+		(effects
+			(font
+				(size 1.27 1.27)
+			)
+			(justify left bottom)
+		)
+	)
+	(label "PH_REF"
 		(at 58.42 60.96 180)
 		(effects
@@
 		)
 	)
-	(label "PH_REF"
-		(at 76.2 139.7 0)
-		(effects
-			(font
-				(size 1.27 1.27)
-			)
-			(justify left bottom)
-		)
-	)
-	(label "AIN2"
-		(at 73.66 205.74 0)
-		(effects
-			(font
-				(size 1.27 1.27)
-			)
-			(justify left bottom)
-		)
-	)
-	(label "AIN3"
-		(at 55.88 245.11 90)
-		(effects
-			(font
-				(size 1.27 1.27)
-			)
-			(justify left bottom)
-		)
-	)

Commit message: kicad: J1 polarity silk (+12V/GND), connector values match aquaPi port names
Terminal values now use the IoRegistry port names (PWM 0/1, GPIO n,
DS1820, ADC #1 in n) instead of the old "OUT G18"-style labels, several of
which were stale after the 74HCT244 reorder. Values stay on F.Fab; only the
J1 polarity marks are added to the silkscreen.

Co-Authored-By: Claude Opus 5.5 <noreply@anthropic.com>
Parts:
- J25: value pH probe -> ADC #1 in 0
- J26: value Module -> ADC #1 in 2
- J27: value AIN3 -> ADC #1 in 3
Changed lines of the file:
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@@
 			)
 		)
-		(property "Value" "AIN3"
+		(property "Value" "ADC #1 in 3"
 			(at 36.576 253.238 0)
 			(show_name no)
@@
 			)
 		)
-		(property "Value" "pH probe"
+		(property "Value" "ADC #1 in 0"
 			(at 29.464 108.204 0)
 			(show_name no)
@@
 			)
 		)
-		(property "Value" "Module"
+		(property "Value" "ADC #1 in 2"
 			(at 38.354 211.328 0)
 			(show_name no)
