File: kicad/analog.kicad_sch (KiCad schematic)
At the start: 23 parts, among them J25 ADC #1 in 0, J26 ADC #1 in 2, J27 ADC #1 in 3, U5 ADS1115IDGSR, U6 TLV9062IDR

Commit message: kicad: schematic re-save (library symbol refresh, BOM field setup)
Parts:
- C13, C15, C16, C17, C18, C19, R45, R46, R47, R48, R49, R50, R51, R52: KiLib_Generator (none) -> SMD_2terminal_chip_molded
- C14: KiLib_Generator (none) -> capacitor/THT/other
- D27, D28, U5, U6: KiLib_Generator (none) -> package/gullwing
- J26, J27: KiLib_Generator (none) -> terminal_block/Phoenix
