File: kicad/outputs.kicad_sch (KiCad schematic)
At the start: 50 parts, among them J4 OUT G18, J5 OUT G19, J6 OUT G12, J7 OUT G13, J8 OUT G16, J9 OUT G26, Q1 AOD4184A, Q2 AOD4184A, Q3 AOD4184A, Q4 AOD4184A, Q5 AOD4184A, Q6 AOD4184A, U3 74HCT244D

Commit message: kicad: restore net names lost while tidying the schematic
27 local labels re-added (Q1-Q6 _OUT/_G/_LED, S1-S4 _OUT/_LED, SSR_V);
the board nets are renamed with all pads and tracks. Connectivity is
unchanged, ERC 0, DRC with schematic parity clean. Q?_OUT match the
"Power" net class pattern again.

Co-Authored-By: Claude Opus 5.5 <noreply@anthropic.com>
Connections:
- net Q5_G: now reaches Q5.1 (G), R26.2, R27.1
- net Q5_OUT: now reaches D14.2 (A), J8.2 (Pin_2), Q5.2 (D)
- net Q6_OUT: now reaches D16.2 (A), J9.2 (Pin_2), Q6.2 (D)
- net Q1_G: now reaches Q1.1 (G), R14.2, R15.1
- net Q2_OUT: now reaches D8.2 (A), J5.2 (Pin_2), Q2.2 (D)
- net Q4_OUT: now reaches D12.2 (A), J7.2 (Pin_2), Q4.2 (D)
- net Q3_OUT: now reaches D10.2 (A), J6.2 (Pin_2), Q3.2 (D)
- net Q3_G: now reaches Q3.1 (G), R20.2, R21.1
- net Q6_G: now reaches Q6.1 (G), R29.2, R30.1
- net Q1_LED: now reaches D7.2 (A), R16.2
- net Q2_G: now reaches Q2.1 (G), R17.2, R18.1
- net Q1_OUT: now reaches D6.2 (A), J4.2 (Pin_2), Q1.2 (D)
- net Q5_LED: now reaches D15.2 (A), R28.2
- net Q4_G: now reaches Q4.1 (G), R23.2, R24.1
- net Q3_LED: now reaches D11.2 (A), R22.2
- net Q2_LED: now reaches D9.2 (A), R19.2
- net Q6_LED: now reaches D17.2 (A), R31.2
- net Q4_LED: now reaches D13.2 (A), R25.2
Changed lines of the file:
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@@
+		)
+	)
+	(label "Q1_OUT"
+		(at 60.96 132.08 0)
+		(effects
+			(font
+				(size 1.27 1.27)
+			)
+			(justify left bottom)
+		)
+	)
+	(label "Q1_G"
+		(at 46.99 123.19 0)
+		(effects
+			(font
+				(size 1.27 1.27)
+			)
+			(justify left bottom)
+		)
+	)
+	(label "Q1_LED"
+		(at 34.29 133.35 0)
+		(effects
+			(font
+				(size 1.27 1.27)
+			)
+			(justify left bottom)
+		)
+	)
+	(label "Q2_OUT"
+		(at 115.57 132.08 0)
+		(effects
+			(font
+				(size 1.27 1.27)
+			)
+			(justify left bottom)
+		)
+	)
+	(label "Q2_G"
+		(at 101.6 123.19 0)
+		(effects
+			(font
+				(size 1.27 1.27)
+			)
+			(justify left bottom)
+		)
+	)
+	(label "Q2_LED"
+		(at 88.9 133.35 0)
+		(effects
+			(font
+				(size 1.27 1.27)
+			)
+			(justify left bottom)
+		)
+	)
+	(label "Q3_OUT"
+		(at 60.96 168.91 0)
+		(effects
+			(font
+				(size 1.27 1.27)
+			)
+			(justify left bottom)
+		)
+	)
+	(label "Q3_G"
+		(at 46.99 160.02 0)
+		(effects
+			(font
+				(size 1.27 1.27)
+			)
+			(justify left bottom)
+		)
+	)
+	(label "Q3_LED"
+		(at 34.29 170.18 0)
+		(effects
+			(font
+				(size 1.27 1.27)
+			)
+			(justify left bottom)
+		)
+	)
+	(label "Q4_OUT"
+		(at 115.57 168.91 0)
+		(effects
+			(font
+				(size 1.27 1.27)
+			)
+			(justify left bottom)
+		)
+	)
+	(label "Q4_G"
+		(at 101.6 160.02 0)
+		(effects
+			(font
+				(size 1.27 1.27)
+			)
+			(justify left bottom)
+		)
+	)
+	(label "Q4_LED"
+		(at 88.9 170.18 0)
+		(effects
+			(font
+				(size 1.27 1.27)
+			)
+			(justify left bottom)
+		)
+	)
+	(label "Q5_OUT"
+		(at 60.96 205.74 0)
+		(effects
+			(font
+				(size 1.27 1.27)
+			)
+			(justify left bottom)
+		)
+	)
+	(label "Q5_G"
+		(at 46.99 196.85 0)
+		(effects
+			(font
+				(size 1.27 1.27)
+			)
+			(justify left bottom)
+		)
+	)
+	(label "Q5_LED"
+		(at 34.29 207.01 0)
+		(effects
+			(font
+				(size 1.27 1.27)
+			)
+			(justify left bottom)
+		)
+	)
+	(label "Q6_OUT"
+		(at 115.57 205.74 0)
+		(effects
+			(font
+				(size 1.27 1.27)
+			)
+			(justify left bottom)
+		)
+	)
+	(label "Q6_G"
+		(at 101.6 196.85 0)
+		(effects
+			(font
+				(size 1.27 1.27)
+			)
+			(justify left bottom)
+		)
+	)
+	(label "Q6_LED"
+		(at 88.9 207.01 0)
+		(effects
+			(font
+				(size 1.27 1.27)
+			)
+			(justify left bottom)
 		)
 	)

Commit message: kicad: reorder 74HCT244 channels for crossing-free Pi -> driver routing
Inputs enter U3 from outside (pull-downs R8..R13 as a staircase), outputs
leave inside under the IC body towards Q1..Q6. The GPIO order on the Pi
header then has to be Q6..Q1, so the stage mapping changes to
Q2 = GPIO12, Q3 = GPIO13, Q4 = GPIO19 (hardware PWM stays on GPIO18/19,
now Q1/Q4). Unused channels: pin 8/11 inputs to GND, pin 9/12 open.

Co-Authored-By: Claude Opus 5.5 <noreply@anthropic.com>
Parts:
- D11: value GPIO12 -> GPIO13
- D13: value GPIO13 -> GPIO19
- D9: value GPIO19 -> GPIO12
Connections:
- net GPIO12_Q3 is gone; now on net GPIO26_Q6: R10.1, U3.6 (1A2)
- net GPIO19_Q2 is gone; now on net GPIO16_Q5: R9.1, U3.4 (1A1)
- net GND: now also U3.8 (1A3); no longer U3.13 (2A2)
- net GPIO16_Q5: no longer R12.1, U3.17 (2A0)
- net GPIO18_Q1: now also R13.1, U3.13 (2A2); no longer R8.1, U3.2 (1A0)
- net GPIO26_Q6: no longer R13.1, U3.15 (2A1)
- net Q1_DRV: now also U3.7 (2Y2); no longer U3.18 (1Y0)
- net Q2_DRV: now also U3.5 (2Y1); no longer U3.16 (1Y1)
- net Q3_DRV: now also U3.3 (2Y0); no longer U3.14 (1Y2)
- net Q4_DRV: now also U3.18 (1Y0); no longer U3.12 (1Y3)
- net Q5_DRV: now also U3.16 (1Y1); no longer U3.3 (2Y0)
- net Q6_DRV: now also U3.14 (1Y2); no longer U3.5 (2Y1)
- net GPIO13_Q4 renamed GPIO13_Q3
- net GPIO13_Q3: now also U3.17 (2A0); no longer U3.8 (1A3)
- new net GPIO12_Q2: R12.1, U3.15 (2A1)
- new net GPIO19_Q4: R8.1, U3.2 (1A0)
Other:
- note added: "Per channel: 100R gate resistor, 10k gate pull-down (off while the Pi boots or is absent), AOD4184A 40 V low-side switch, SS54 freewheel diode to VIN, status LED on the 5 V drive signal. Q1/Q4 = hardware PWM (GPIO18/19: light, fan). Terminal: pin 1 = +VIN, pin 2 = switched OUT (load between)."
- note removed: "Per channel: 100R gate resistor, 10k gate pull-down (off while the Pi boots or is absent), AOD4184A 40 V low-side switch, SS54 freewheel diode to VIN, status LED on the 5 V drive signal. Q1/Q2 = hardware PWM (light, fan). Terminal: pin 1 = +VIN, pin 2 = switched OUT (load between)."
Changed lines of the file:
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@@
 		(comment 1 "CERN-OHL-S-2.0")
 	)
-	(text "Per channel: 100R gate resistor, 10k gate pull-down (off while the Pi boots or is absent),\nAOD4184A 40 V low-side switch, SS54 freewheel diode to VIN, status LED on the 5 V drive signal.\nQ1/Q2 = hardware PWM (light, fan). Terminal: pin 1 = +VIN, pin 2 = switched OUT (load between)."
+	(text "Per channel: 100R gate resistor, 10k gate pull-down (off while the Pi boots or is absent),\nAOD4184A 40 V low-side switch, SS54 freewheel diode to VIN, status LED on the 5 V drive signal.\nQ1/Q4 = hardware PWM (GPIO18/19: light, fan). Terminal: pin 1 = +VIN, pin 2 = switched OUT (load between)."
 		(exclude_from_sim no)
 		(at 25.4 109.22 0)
@@
 	)
 	(junction
-		(at 38.1 71.12)
-		(diameter 0)
-		(color 0 0 0 0)
-	)
-	(junction
 		(at 101.6 210.82)
 		(diameter 0)
@@
 	)
 	(no_connect
-		(at 66.04 68.58)
+		(at 66.04 60.96)
 	)
 	(wire
@@
 	(wire
 		(pts
-			(xy 66.04 60.96) (xy 68.58 60.96)
+			(xy 66.04 68.58) (xy 68.58 68.58)
 		)
 		(stroke
@@
 	(wire
 		(pts
-			(xy 38.1 68.58) (xy 38.1 71.12)
-		)
-		(stroke
-			(width 0)
-			(type default)
-		)
-	)
-	(wire
-		(pts
 			(xy 46.99 134.62) (xy 53.34 134.62)
 		)
@@
 		)
 	)
-	(label "Q6_DRV"
+	(label "Q2_DRV"
 		(at 68.58 66.04 0)
 		(effects
@@
 		)
 	)
-	(label "Q4_DRV"
-		(at 68.58 60.96 0)
+	(label "Q1_DRV"
+		(at 68.58 68.58 0)
 		(effects
 			(font
@@
 		)
 	)
-	(label "Q2_DRV"
+	(label "Q5_DRV"
 		(at 68.58 55.88 0)
 		(effects
@@
 		)
 	)
-	(label "Q5_DRV"
+	(label "Q3_DRV"
 		(at 68.58 63.5 0)
 		(effects
@@
 		)
 	)
-	(label "Q1_DRV"
+	(label "Q4_DRV"
 		(at 68.58 53.34 0)
 		(effects
@@
 		)
 	)
-	(label "Q3_DRV"
+	(label "Q6_DRV"
 		(at 68.58 58.42 0)
 		(effects
@@
 		)
 	)
-	(global_label "GPIO26_Q6"
+	(global_label "GPIO18_Q1"
 		(shape bidirectional)
 		(at 153.67 59.69 90)
@@
 		)
 	)
-	(global_label "GPIO12_Q3"
+	(global_label "GPIO26_Q6"
 		(shape bidirectional)
 		(at 123.19 59.69 90)
@@
 		)
 	)
-	(global_label "GPIO16_Q5"
+	(global_label "GPIO13_Q3"
 		(shape bidirectional)
 		(at 38.1 63.5 180)
@@
 		)
 	)
-	(global_label "GPIO19_Q2"
+	(global_label "GPIO16_Q5"
 		(shape bidirectional)
 		(at 111.76 59.69 90)
@@
 		)
 	)
-	(global_label "GPIO13_Q4"
+	(global_label "GPIO18_Q1"
 		(shape bidirectional)
-		(at 38.1 60.96 180)
+		(at 38.1 68.58 180)
 		(fields_autoplaced yes)
 		(effects
@@
 		)
 		(property "Intersheetrefs" "${INTERSHEET_REFS}"
-			(at 38.1 60.96 0)
+			(at 38.1 68.58 0)
 			(hide yes)
 			(show_name no)
@@
 		)
 	)
-	(global_label "GPIO12_Q3"
+	(global_label "GPIO26_Q6"
 		(shape bidirectional)
 		(at 38.1 58.42 180)
@@
 		)
 	)
-	(global_label "GPIO26_Q6"
+	(global_label "GPIO12_Q2"
 		(shape bidirectional)
 		(at 38.1 66.04 180)
@@
 		)
 	)
-	(global_label "GPIO19_Q2"
+	(global_label "GPIO16_Q5"
 		(shape bidirectional)
 		(at 38.1 55.88 180)
@@
 		)
 	)
-	(global_label "GPIO18_Q1"
+	(global_label "GPIO19_Q4"
 		(shape bidirectional)
 		(at 100.33 59.69 90)
@@
 		)
 	)
-	(global_label "GPIO13_Q4"
+	(global_label "GPIO13_Q3"
 		(shape bidirectional)
 		(at 133.35 59.69 90)
@@
 		)
 	)
-	(global_label "GPIO16_Q5"
+	(global_label "GPIO12_Q2"
 		(shape bidirectional)
 		(at 143.51 59.69 90)
@@
 		)
 	)
-	(global_label "GPIO18_Q1"
+	(global_label "GPIO19_Q4"
 		(shape bidirectional)
 		(at 38.1 53.34 180)
@@
 		)
 	)
+		(symbol
+		(lib_id "power:GND")
+		(at 38.1 60.96 270)
+		(unit 1)
+		(body_style 1)
+		(exclude_from_sim no)
+		(in_bom no)
+		(on_board no)
+		(in_pos_files yes)
+		(dnp no)
+		(property "Reference" "#PWR164"
+			(at 31.75 60.96 0)
+			(hide yes)
+			(show_name no)
+			(do_not_autoplace no)
+			(effects
+				(font
+					(size 1.27 1.27)
+				)
+			)
+		)
+		(property "Value" "GND"
+			(at 34.29 60.96 0)
+			(hide yes)
+			(show_name no)
+			(do_not_autoplace no)
+			(effects
+				(font
+					(size 1.27 1.27)
+				)
+			)
+		)
+		(property "Footprint" ""
+			(at 38.1 60.96 0)
+			(hide yes)
+			(show_name no)
+			(do_not_autoplace no)
+			(effects
+				(font
+					(size 1.27 1.27)
+				)
+			)
+		)
+		(property "Datasheet" ""
+			(at 38.1 60.96 0)
+			(hide yes)
+			(show_name no)
+			(do_not_autoplace no)
+			(effects
+				(font
+					(size 1.27 1.27)
+				)
+			)
+		)
+		(property "Description" "Power symbol creates a global label with name \"GND\" , ground"
+			(at 38.1 60.96 0)
+			(hide yes)
+			(show_name no)
+			(do_not_autoplace no)
+			(effects
+				(font
+					(size 1.27 1.27)
+				)
+			)
+		)
+		(pin "1"
+		)
+		(instances
+			(project "aquaPCB"
+				(path "/80232f81-1179-4777-a7f0-674a974d53cc/662aa388-f80b-440b-be99-bc584ab7592b"
+					(reference "#PWR164")
+					(unit 1)
+				)
+			)
+		)
+	)
 	(symbol
 		(lib_id "Device:R")
@@
 			)
 		)
-		(property "Value" "GPIO19"
+		(property "Value" "GPIO12"
 			(at 94.234 145.542 90)
 			(show_name no)
@@
 			)
 		)
-		(property "Value" "GPIO13"
+		(property "Value" "GPIO19"
 			(at 94.361 182.499 90)
 			(show_name no)
@@
 			)
 		)
-		(property "Value" "GPIO12"
+		(property "Value" "GPIO13"
 			(at 39.878 182.372 90)
 			(show_name no)

Commit message: kicad: J1 polarity silk (+12V/GND), connector values match aquaPi port names
Terminal values now use the IoRegistry port names (PWM 0/1, GPIO n,
DS1820, ADC #1 in n) instead of the old "OUT G18"-style labels, several of
which were stale after the 74HCT244 reorder. Values stay on F.Fab; only the
J1 polarity marks are added to the silkscreen.

Co-Authored-By: Claude Opus 5.5 <noreply@anthropic.com>
Parts:
- J4: value OUT G18 -> PWM 0
- J5: value OUT G19 -> GPIO 12
- J6: value OUT G12 -> GPIO 13
- J7: value OUT G13 -> PWM 1
- J8: value OUT G16 -> GPIO 16
- J9: value OUT G26 -> GPIO 26
Changed lines of the file:
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@@
 			)
 		)
-		(property "Value" "OUT G26"
+		(property "Value" "GPIO 26"
 			(at 129.794 208.534 0)
 			(show_name no)
@@
 			)
 		)
-		(property "Value" "OUT G16"
+		(property "Value" "GPIO 16"
 			(at 74.676 208.788 0)
 			(show_name no)
@@
 			)
 		)
-		(property "Value" "OUT G12"
+		(property "Value" "GPIO 13"
 			(at 76.454 171.958 0)
 			(show_name no)
@@
 			)
 		)
-		(property "Value" "OUT G19"
+		(property "Value" "GPIO 12"
 			(at 130.048 135.128 0)
 			(show_name no)
@@
 			)
 		)
-		(property "Value" "OUT G18"
+		(property "Value" "PWM 0"
 			(at 75.692 135.128 0)
 			(show_name no)
@@
 			)
 		)
-		(property "Value" "OUT G13"
+		(property "Value" "PWM 1"
 			(at 129.286 171.704 0)
 			(show_name no)
