File: kicad/outputs.kicad_sch (KiCad schematic)
At the start: 50 parts, among them J4 PWM 0, J5 GPIO 12, J6 GPIO 13, J7 PWM 1, J8 GPIO 16, J9 GPIO 26, Q1 AOD4184A, Q2 AOD4184A, Q3 AOD4184A, Q4 AOD4184A, Q5 AOD4184A, Q6 AOD4184A, U3 74HCT244D

Commit message: kicad: schematic re-save (library symbol refresh, BOM field setup)
Parts:
- C12, D11, D13, D15, D17, D7, D9, R10, R11, R12, R13, R14, R15, R16, R17, R18, R19, R20, R21, R22, R23, R24, R25, R26, R27, R28, R29, R30, R31, R8, R9: KiLib_Generator (none) -> SMD_2terminal_chip_molded
- J4, J5, J6, J7, J8, J9: KiLib_Generator (none) -> terminal_block/Phoenix
- Q1, Q2, Q3, Q4, Q5, Q6: KiLib_Generator (none) -> package/TO_SOT/SMD
- U3: KiLib_Generator (none) -> package/gullwing
