File: kicad/outputs.kicad_sch (KiCad schematic)
At the start: 50 parts, among them J4 PWM 0, J5 GPIO 12, J6 GPIO 13, J7 PWM 1, J8 GPIO 16, J9 GPIO 26, Q1 AOD4184A, Q2 AOD4184A, Q3 AOD4184A, Q4 AOD4184A, Q5 AOD4184A, Q6 AOD4184A, U3 74HCT244D

Commit message: kicad: v2 schematic and board update (PCA9685 x2, box-header ports, sensors, analog sockets)
New sheets pwm/powerbar/sensors; Q2/3/5/6 on PCA #1 ch 15-12; sensor GPIOs 5,6,20,21,22,23; 1-Wire +5V_EXT/Data/GND; four identical 0-5 V analog sockets; DC/LED/sensor ports as 2x4 box headers (pin n = Robo-Tank v3 RJ45 pin n). Board: 82 new footprints coarse-placed (56 parked beside the board), ERC 0, DRC copper 0, parity 0. README v2 plan updated.

Co-Authored-By: Claude Opus 5.5 <noreply@anthropic.com>
Connections:
- net GPIO12_Q2 renamed PCA1_CH15
- net GPIO13_Q3 renamed PCA1_CH14
- net GPIO16_Q5 renamed PCA1_CH13
- net GPIO26_Q6 renamed PCA1_CH12
Changed lines of the file:
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@@
 		)
 	)
-	(global_label "GPIO26_Q6"
+	(global_label "PCA1_CH12"
 		(shape bidirectional)
 		(at 123.19 59.69 90)
@@
 		)
 	)
-	(global_label "GPIO13_Q3"
+	(global_label "PCA1_CH14"
 		(shape bidirectional)
 		(at 38.1 63.5 180)
@@
 		)
 	)
-	(global_label "GPIO16_Q5"
+	(global_label "PCA1_CH13"
 		(shape bidirectional)
 		(at 111.76 59.69 90)
@@
 		)
 	)
-	(global_label "GPIO26_Q6"
+	(global_label "PCA1_CH12"
 		(shape bidirectional)
 		(at 38.1 58.42 180)
@@
 		)
 	)
-	(global_label "GPIO12_Q2"
+	(global_label "PCA1_CH15"
 		(shape bidirectional)
 		(at 38.1 66.04 180)
@@
 		)
 	)
-	(global_label "GPIO16_Q5"
+	(global_label "PCA1_CH13"
 		(shape bidirectional)
 		(at 38.1 55.88 180)
@@
 		)
 	)
-	(global_label "GPIO13_Q3"
+	(global_label "PCA1_CH14"
 		(shape bidirectional)
 		(at 133.35 59.69 90)
@@
 		)
 	)
-	(global_label "GPIO12_Q2"
+	(global_label "PCA1_CH15"
 		(shape bidirectional)
 		(at 143.51 59.69 90)

Commit message: kicad: v2 layout finished - ADC renumbering, port labels, last routes
- ADC sockets numbered 0..3 from right to left; AIN0<->AIN1 and AIN2<->AIN3
  swapped at the ADS1115, U5 end runs re-routed.
- Connector labels: IoRegistry-style port names (PCA#1 chNN, ADC #1 in n,
  GPIO n, DS1820); J5/J6/J8/J9 corrected from GPIO to PCA#1 ch15/14/13/12
  (also in outputs.kicad_sch). Back side: names with voltage/current
  ratings, running from the board edge at pin 1, "+" on supply pins,
  SCL/SDA and 1-Wire Data marks. Front: ADC #1 / in n, jumper labels.
- Routed the last six open nets (+3V3 at J24/JP4, +5V_EXT at J19,
  GPIO2_SDA J22-J23 on B.Cu, AIN1, J24 pin 10 - JP3, PCA1_CH1); PCA1_CH3
  partly moved to B.Cu to free the corridor at U7. Dangling stubs removed.
- Silkscreen: nothing on pads, overlaps reduced with small moves; part
  references and F.Fab texts at 0.8 mm.
- aquaPCB.kicad_dru: the deliberate courtyard overlap of the ADC socket
  pairs J26/J27 and J36/J37 (2.54 mm grid) is waived by a custom rule.

ERC clean, DRC without errors (silkscreen warnings only), board fully
routed and in sync with the schematic.

Co-Authored-By: Claude Opus 5.5 <noreply@anthropic.com>
Parts:
- J5: value GPIO 12 -> PCA#1 ch15
- J6: value GPIO 13 -> PCA#1 ch14
- J8: value GPIO 16 -> PCA#1 ch13
- J9: value GPIO 26 -> PCA#1 ch12
Changed lines of the file:
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@@
 			)
 		)
-		(property "Value" "GPIO 26"
+		(property "Value" "PCA#1 ch12"
 			(at 129.794 208.534 0)
 			(show_name no)
@@
 			)
 		)
-		(property "Value" "GPIO 16"
+		(property "Value" "PCA#1 ch13"
 			(at 74.676 208.788 0)
 			(show_name no)
@@
 			)
 		)
-		(property "Value" "GPIO 13"
+		(property "Value" "PCA#1 ch14"
 			(at 76.454 171.958 0)
 			(show_name no)
@@
 			)
 		)
-		(property "Value" "GPIO 12"
+		(property "Value" "PCA#1 ch15"
 			(at 130.048 135.128 0)
 			(show_name no)

Commit message: kicad: LCSC numbers for PCA9685 and PTC, status LED names follow PCA#1
- U7/U10 PCA9685PW,118 -> LCSC C2678753, F2 nSMD050 -> C69688 (schematic
  and board), so every assembled part carries an LCSC number.
- Status LEDs D9/D11/D15/D17 renamed GPIO12/13/16/26 -> PCA#1 ch15/14/13/12,
  matching the Q2/Q3/Q5/Q6 drive since v2.

Co-Authored-By: Claude Opus 5.5 <noreply@anthropic.com>
Parts:
- D11: value GPIO13 -> PCA#1 ch14
- D15: value GPIO16 -> PCA#1 ch13
- D17: value GPIO26 -> PCA#1 ch12
- D9: value GPIO12 -> PCA#1 ch15
Changed lines of the file:
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@@
 			)
 		)
-		(property "Value" "GPIO16"
+		(property "Value" "PCA#1 ch13"
 			(at 39.37 221.742 90)
 			(show_name no)
@@
 			)
 		)
-		(property "Value" "GPIO12"
+		(property "Value" "PCA#1 ch15"
 			(at 94.234 145.542 90)
 			(show_name no)
@@
 			)
 		)
-		(property "Value" "GPIO26"
+		(property "Value" "PCA#1 ch12"
 			(at 94.361 221.869 90)
 			(show_name no)
@@
 			)
 		)
-		(property "Value" "GPIO13"
+		(property "Value" "PCA#1 ch14"
 			(at 39.878 182.372 90)
 			(show_name no)
