File: kicad/power.kicad_sch (KiCad schematic)
At the start: 30 parts, among them J1 12V IN, Q10 AOD4185, U1 TPS54360B, U2 AMS1117-3.3

Commit message: kicad: push-in spring terminals (Kangnex WJ250B), 8 A total
All 18 screw terminals replaced by Ningbo Kangnex WJ250B push-in spring
terminals (LCSC C8454 2-pole, C8420 3-pole; 3.5 mm pitch, staggered
pins, 8 A IEC). New footprints from the EasyEDA pad data and the maker
drawing (wire entry on the pin-1 side, facing the board edge) and
simple 3D models. Board total current reduced to 8 A: fuse 8 A
(Littelfuse 0154008.DR, LCSC C206919). Board: footprints swapped with
nets and schematic links kept, edges re-placed for the deeper bodies.
ERC 0; DRC unchanged (known J2/Zero-hole overlap, silk, unrouted).
Docs: BOM/README (8 A budget, 5.3 mm input path, cost ~35 EUR/board).

Co-Authored-By: Claude Opus 5.5 <noreply@anthropic.com>
Parts:
- F1: value 10A -> 8A; LCSC (none) -> C206919; Reichelt LITT 0154010.DR -> (none)
- J1: footprint TerminalBlock_Phoenix:TerminalBlock_Phoenix_MKDS-1,5-2-5.08_1x02_P5.08mm_Horizontal -> aquaPCB:TerminalBlock_Kangnex_WJ250B-3.5-02P_P3.50mm_Staggered; LCSC (none) -> C8454; Reichelt AKL 101-02 -> (none)
Changed lines of the file:
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@@
 			)
 		)
-		(property "Footprint" "TerminalBlock_Phoenix:TerminalBlock_Phoenix_MKDS-1,5-2-5.08_1x02_P5.08mm_Horizontal"
+		(property "Footprint" "aquaPCB:TerminalBlock_Kangnex_WJ250B-3.5-02P_P3.50mm_Staggered"
 			(at 48.26 72.39 0)
 			(hide yes)
@@
 			)
 		)
-		(property "Reichelt" "AKL 101-02"
+		(property "LCSC" "C8454"
 			(at 48.26 72.39 0)
 			(hide yes)
@@
 			)
 		)
-		(property "Value" "10A"
+		(property "Value" "8A"
 			(at 66.04 59.69 0)
 			(show_name no)
@@
 			)
 		)
-		(property "Reichelt" "LITT 0154010.DR"
+		(property "LCSC" "C206919"
 			(at 69.85 59.69 0)
 			(hide yes)

Commit message: kicad: routing progress (by hand)
Co-Authored-By: Claude Opus 5.5 (1M context) <noreply@anthropic.com>
Parts:
- D3: value LED red -> PWR, red
- D5: value LED green -> 3V3, green
Other:
- moved on the sheet: C2, C3, C4, C5, C6, C7, C8, C9, D4, JP1, L1, R3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

Commit message: kicad: swap J1 pins (pin 1 = GND), remove floating GND islands
J1 GND now sits on the lower pole, so the ground plane leaves the input
terminal directly east towards Q1..Q6 instead of being boxed in by the
VIN_RAW B.Cu feed. VIN_RAW now starts at the upper pole (3 mm on both
layers as before). Schematic: J1 rotated 180 deg instead of mirrored, wiring
unchanged. GND B.Cu zone island removal set to "always" (removes the
floating 1.05 mm2 island next to J1).

Co-Authored-By: Claude Opus 5.5 <noreply@anthropic.com>
Connections:
- net GND: now also J1.1 (Pin_1); no longer J1.2 (Pin_2)
- net VIN_RAW: now also J1.2 (Pin_2); no longer J1.1 (Pin_1)
Other:
- moved on the sheet: J1
Changed lines of the file:
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@@
 	(symbol
 		(lib_id "Connector:Screw_Terminal_01x02")
-		(at 48.26 72.39 0)
-		(mirror y)
+		(at 48.26 74.93 180)
 		(unit 1)
 		(body_style 1)

Commit message: kicad: shorten D3/D5 values in schematic to match the board (PWR, 3V3)
Co-Authored-By: Claude Opus 5.5 <noreply@anthropic.com>
Parts:
- D3: value PWR, red -> PWR
- D5: value 3V3, green -> 3V3
Changed lines of the file:
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@@
 			)
 		)
-		(property "Value" "3V3, green"
+		(property "Value" "3V3"
 			(at 143.51 223.266 90)
 			(show_name no)
@@
 			)
 		)
-		(property "Value" "PWR, red"
+		(property "Value" "PWR"
 			(at 138.43 81.534 90)
 			(show_name no)
