File: kicad/power.kicad_sch (KiCad schematic)
At the start: 30 parts, among them J1 12V IN, Q10 AOD4185, U1 TPS54360B, U2 AMS1117-3.3

Commit message: kicad: schematic re-save (library symbol refresh, BOM field setup)
Parts:
- C1: KiLib_Generator (none) -> capacitor/THT/other
- C10, C11, C2, C3, C4, C5, C6, C7, C8, C9, D3, D5, R1, R2, R3, R4, R5, R6, R7: KiLib_Generator (none) -> SMD_2terminal_chip_molded
- J1: KiLib_Generator (none) -> terminal_block/Phoenix
- JP1: KiLib_Generator (none) -> connector/pin_header_socket
- L1: KiLib_Generator (none) -> inductor/SMD
- Q10: KiLib_Generator (none) -> package/TO_SOT/SMD
