File: kicad/power.kicad_sch (KiCad schematic)
At the start: 30 parts, among them J1 12V IN, Q10 AOD4185, U1 TPS54360B, U2 AMS1117-3.3

Commit message: kicad: pin headers for 1-Wire, ADC and floats; connectivity-driven re-placement
J19, ADC sockets (J36/J37/J26/J27, 3x4 grid) and floats J30/J31 are pin headers now. All footprints placed on the board (big connectors first, flat parts allowed under the Pi, user-placed U10/RN5/J32/U11 and user routing kept): signal ratsnest 7824 -> 4450 mm, crossings 1776 -> 862. ERC 0, DRC copper 0, parity 0.

Co-Authored-By: Claude Opus 5.5 <noreply@anthropic.com>
Parts:
- added C24, C25: 10u, Capacitor_SMD:C_0603_1608Metric, symbol Device:C
- added U11: AMS1117-3.3, Package_TO_SOT_SMD:SOT-223-3_TabPin2, symbol Regulator_Linear:AMS1117-3.3
Connections:
- net GND: now also C24.2, C25.2, U11.1 (GND)
- new net +3V3_EXT: C25.1, U11.2 (VO)
- new net +5V_EXT: C24.1, U11.3 (VI)
Other:
- note added: "+3V3_EXT: separate 3.3 V for external loads (feeder on power bar header pin 10), keeps motor noise off the +3V3 rail of ADS1115 / PCA9685"

Commit message: kicad: v2 layout finished - ADC renumbering, port labels, last routes
- ADC sockets numbered 0..3 from right to left; AIN0<->AIN1 and AIN2<->AIN3
  swapped at the ADS1115, U5 end runs re-routed.
- Connector labels: IoRegistry-style port names (PCA#1 chNN, ADC #1 in n,
  GPIO n, DS1820); J5/J6/J8/J9 corrected from GPIO to PCA#1 ch15/14/13/12
  (also in outputs.kicad_sch). Back side: names with voltage/current
  ratings, running from the board edge at pin 1, "+" on supply pins,
  SCL/SDA and 1-Wire Data marks. Front: ADC #1 / in n, jumper labels.
- Routed the last six open nets (+3V3 at J24/JP4, +5V_EXT at J19,
  GPIO2_SDA J22-J23 on B.Cu, AIN1, J24 pin 10 - JP3, PCA1_CH1); PCA1_CH3
  partly moved to B.Cu to free the corridor at U7. Dangling stubs removed.
- Silkscreen: nothing on pads, overlaps reduced with small moves; part
  references and F.Fab texts at 0.8 mm.
- aquaPCB.kicad_dru: the deliberate courtyard overlap of the ADC socket
  pairs J26/J27 and J36/J37 (2.54 mm grid) is waived by a custom rule.

ERC clean, DRC without errors (silkscreen warnings only), board fully
routed and in sync with the schematic.

Co-Authored-By: Claude Opus 5.5 <noreply@anthropic.com>
Parts:
- C24, C25: footprint Capacitor_SMD:C_0603_1608Metric -> Capacitor_SMD:C_0805_2012Metric; LCSC C19702 -> C15850
Changed lines of the file:
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@@
 			)
 		)
-		(property "Footprint" "Capacitor_SMD:C_0603_1608Metric"
+		(property "Footprint" "Capacitor_SMD:C_0805_2012Metric"
 			(at 72.39 264.16 0)
 			(hide yes)
@@
 			)
 		)
-		(property "LCSC" "C19702"
+		(property "LCSC" "C15850"
 			(at 72.39 264.16 0)
 			(hide yes)
@@
 			)
 		)
-		(property "Footprint" "Capacitor_SMD:C_0603_1608Metric"
+		(property "Footprint" "Capacitor_SMD:C_0805_2012Metric"
 			(at 80.01 265.43 0)
 			(hide yes)
@@
 			)
 		)
-		(property "LCSC" "C19702"
+		(property "LCSC" "C15850"
 			(at 80.01 265.43 0)
 			(hide yes)

Commit message: kicad: current paths and thermal fixes in the power section
- 10 VIN vias at the Q10 source (was 6); SW node and 5V_PI widened to 1.5 mm;
  F1 -> Q10 drain widened to 5.5 mm.
- J1 GND pads: local thermal spoke width 1.0 mm (7 spokes into the B.Cu GND plane).
- Q10 drain copper zone (Q10_DRAIN, F.Cu, ~1.25 cm2) for Q10 and the fuse holder.
- Q10 AOD4185 -> DMP4010SK3Q-13 (9.9 mOhm, same DPAK pinout); F1 8 A -> 10 A insert
  (0154010.DR, same holder); F2 PTC 0.5 A -> nSMD110 (1.1 A hold) since the feeder
  shares +5V_EXT.
- B.Cu solder mask opening over the VIN trunk to J4 (optional hand tinning).
- Silkscreen: "max 5A, total 6.5A" on both sides; "12V IN" label nudged off the opening.

ERC clean, DRC without errors, board in sync with the schematic.

Co-Authored-By: Claude Opus 5.5 <noreply@anthropic.com>
Parts:
- F1: value 8A -> 10A; LCSC C206919 -> C206921
- Q10: value AOD4185 -> DMP4010SK3Q; LCSC C400894 -> C5359358
Changed lines of the file:
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@@
 			)
 		)
-		(property "Value" "8A"
+		(property "Value" "10A"
 			(at 66.04 59.69 0)
 			(show_name no)
@@
 			)
 		)
-		(property "LCSC" "C206919"
+		(property "LCSC" "C206921"
 			(at 69.85 59.69 0)
 			(hide yes)
@@
 			)
 		)
-		(property "Value" "AOD4185"
+		(property "Value" "DMP4010SK3Q"
 			(at 90.17 56.896 90)
 			(show_name no)
@@
 			)
 		)
-		(property "LCSC" "C400894"
+		(property "LCSC" "C5359358"
 			(at 85.09 54.61 0)
 			(hide yes)
