File: kicad/io.kicad_sch (KiCad schematic)
At the start: 24 parts, among them J15 IN1, J16 IN2, J17 IN3, J18 IN4, J19 1-Wire 1, J20 1-Wire 2, J22 I2C 1, J23 I2C 2, J24 Display

Commit message: kicad: drop UART console and second 1-Wire terminal, tighten buck loop
Schematic: J3 (UART console) and J20 (1-Wire 2) removed by minimal
edits; Pi header pins 8/10 (GPIO14/15) marked no-connect. ERC clean,
connectivity otherwise unchanged.
Board: J3/J20 removed, S1-S4 moved up on the right edge, buck converter
placed per TI layout guidance (D4 SW pad 2.8 mm and L1 SW pad 3.7 mm
from U1-SW, input cap 3.5 mm from VIN, control parts away from SW;
>= 25.9 mm to the pH input). DRC with schematic parity: only the known
J2/Zero-hole overlap, silkscreen and unrouted nets.
Docs: 1 AKL 101-03 less, 35 header pins, cost ~40 EUR/board at 5.

Co-Authored-By: Claude Opus 5.5 <noreply@anthropic.com>
Parts:
- removed J20: 1-Wire 2, TerminalBlock_Phoenix:TerminalBlock_Phoenix_MKDS-1,5-3-5.08_1x03_P5.08mm_Horizontal, symbol Connector:Screw_Terminal_01x03

Commit message: kicad: mark optional headers as DNP
J10 (ULN spare), J23 (2nd I2C), J24 (display) and JP3 (backlight) get
the Do-Not-Populate flag in schematic and board. Footprints stay; BOM
and pick-and-place exports with --exclude-dnp leave them out (checked:
150 -> 146 parts). ERC clean, DRC unchanged. README: new "Build
options" section; BOM: header/jumper counts.

Co-Authored-By: Claude Opus 5.5 <noreply@anthropic.com>
Parts:
- J23, J24, JP3: now not fitted
Changed lines of the file:
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@@
 		(on_board yes)
 		(in_pos_files yes)
-		(dnp no)
+		(dnp yes)
 		(property "Reference" "J24"
 			(at 36.322 233.172 0)
@@
 		(on_board yes)
 		(in_pos_files yes)
-		(dnp no)
+		(dnp yes)
 		(property "Reference" "J23"
 			(at 34.036 179.07 0)
@@
 		(on_board yes)
 		(in_pos_files yes)
-		(dnp no)
+		(dnp yes)
 		(property "Reference" "JP3"
 			(at 45.212 232.664 0)

Commit message: kicad: push-in spring terminals (Kangnex WJ250B), 8 A total
All 18 screw terminals replaced by Ningbo Kangnex WJ250B push-in spring
terminals (LCSC C8454 2-pole, C8420 3-pole; 3.5 mm pitch, staggered
pins, 8 A IEC). New footprints from the EasyEDA pad data and the maker
drawing (wire entry on the pin-1 side, facing the board edge) and
simple 3D models. Board total current reduced to 8 A: fuse 8 A
(Littelfuse 0154008.DR, LCSC C206919). Board: footprints swapped with
nets and schematic links kept, edges re-placed for the deeper bodies.
ERC 0; DRC unchanged (known J2/Zero-hole overlap, silk, unrouted).
Docs: BOM/README (8 A budget, 5.3 mm input path, cost ~35 EUR/board).

Co-Authored-By: Claude Opus 5.5 <noreply@anthropic.com>
Parts:
- J15, J16, J17, J18, J19: footprint TerminalBlock_Phoenix:TerminalBlock_Phoenix_MKDS-1,5-3-5.08_1x03_P5.08mm_Horizontal -> aquaPCB:TerminalBlock_Kangnex_WJ250B-3.5-03P_P3.50mm_Staggered; LCSC (none) -> C8420; Reichelt AKL 101-03 -> (none)
Changed lines of the file:
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@@
 			)
 		)
-		(property "Footprint" "TerminalBlock_Phoenix:TerminalBlock_Phoenix_MKDS-1,5-3-5.08_1x03_P5.08mm_Horizontal"
+		(property "Footprint" "aquaPCB:TerminalBlock_Kangnex_WJ250B-3.5-03P_P3.50mm_Staggered"
 			(at 101.6 49.53 0)
 			(hide yes)
@@
 			)
 		)
-		(property "Reichelt" "AKL 101-03"
+		(property "LCSC" "C8420"
 			(at 101.6 49.53 0)
 			(hide yes)
@@
 			)
 		)
-		(property "Footprint" "TerminalBlock_Phoenix:TerminalBlock_Phoenix_MKDS-1,5-3-5.08_1x03_P5.08mm_Horizontal"
+		(property "Footprint" "aquaPCB:TerminalBlock_Kangnex_WJ250B-3.5-03P_P3.50mm_Staggered"
 			(at 31.75 49.53 0)
 			(hide yes)
@@
 			)
 		)
-		(property "Reichelt" "AKL 101-03"
+		(property "LCSC" "C8420"
 			(at 31.75 49.53 0)
 			(hide yes)
@@
 			)
 		)
-		(property "Footprint" "TerminalBlock_Phoenix:TerminalBlock_Phoenix_MKDS-1,5-3-5.08_1x03_P5.08mm_Horizontal"
+		(property "Footprint" "aquaPCB:TerminalBlock_Kangnex_WJ250B-3.5-03P_P3.50mm_Staggered"
 			(at 101.6 80.01 0)
 			(hide yes)
@@
 			)
 		)
-		(property "Reichelt" "AKL 101-03"
+		(property "LCSC" "C8420"
 			(at 101.6 80.01 0)
 			(hide yes)
@@
 			)
 		)
-		(property "Footprint" "TerminalBlock_Phoenix:TerminalBlock_Phoenix_MKDS-1,5-3-5.08_1x03_P5.08mm_Horizontal"
+		(property "Footprint" "aquaPCB:TerminalBlock_Kangnex_WJ250B-3.5-03P_P3.50mm_Staggered"
 			(at 31.75 80.01 0)
 			(hide yes)
@@
 			)
 		)
-		(property "Reichelt" "AKL 101-03"
+		(property "LCSC" "C8420"
 			(at 31.75 80.01 0)
 			(hide yes)
@@
 			)
 		)
-		(property "Footprint" "TerminalBlock_Phoenix:TerminalBlock_Phoenix_MKDS-1,5-3-5.08_1x03_P5.08mm_Horizontal"
+		(property "Footprint" "aquaPCB:TerminalBlock_Kangnex_WJ250B-3.5-03P_P3.50mm_Staggered"
 			(at 33.02 120.65 0)
 			(hide yes)
@@
 			)
 		)
-		(property "Reichelt" "AKL 101-03"
+		(property "LCSC" "C8420"
 			(at 33.02 120.65 0)
 			(hide yes)

Commit message: kicad: routing progress (by hand)
Co-Authored-By: Claude Opus 5.5 (1M context) <noreply@anthropic.com>
Changed lines of the file:
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@@
 	(generator "eeschema")
 	(generator_version "10.0")
-	(paper "A3")
+	(paper "A4" portrait)
 	(title_block
 		(title "aquaPCB – Inputs, 1-Wire, I2C and display headers")
@@
 	)
 	(junction
-		(at 46.99 120.65)
-		(diameter 0)
-		(color 0 0 0 0)
-	)
-	(junction
 		(at 142.24 80.01)
 		(diameter 0)
@@
 	(wire
 		(pts
-			(xy 38.1 120.65) (xy 46.99 120.65)
+			(xy 38.1 120.65) (xy 57.15 120.65)
 		)
 		(stroke
@@
 		)
 		(stroke
-			(width 0)
-			(type default)
-		)
-	)
-	(wire
-		(pts
-			(xy 46.99 120.65) (xy 57.15 120.65)
-		)
-		(stroke

Commit message: kicad: J1 polarity silk (+12V/GND), connector values match aquaPi port names
Terminal values now use the IoRegistry port names (PWM 0/1, GPIO n,
DS1820, ADC #1 in n) instead of the old "OUT G18"-style labels, several of
which were stale after the 74HCT244 reorder. Values stay on F.Fab; only the
J1 polarity marks are added to the silkscreen.

Co-Authored-By: Claude Opus 5.5 <noreply@anthropic.com>
Parts:
- J15: value IN1 -> GPIO 5
- J16: value IN2 -> GPIO 6
- J17: value IN3 -> GPIO 20
- J18: value IN4 -> GPIO 21
- J19: value 1-Wire 1 -> DS1820
Changed lines of the file:
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@@
 			)
 		)
-		(property "Value" "IN3"
+		(property "Value" "GPIO 20"
 			(at 102.616 54.864 0)
 			(show_name no)
@@
 			)
 		)
-		(property "Value" "IN1"
+		(property "Value" "GPIO 5"
 			(at 32.258 55.626 0)
 			(show_name no)
@@
 			)
 		)
-		(property "Value" "IN4"
+		(property "Value" "GPIO 21"
 			(at 102.362 85.598 0)
 			(show_name no)
@@
 			)
 		)
-		(property "Value" "IN2"
+		(property "Value" "GPIO 6"
 			(at 32.512 85.598 0)
 			(show_name no)
@@
 			)
 		)
-		(property "Value" "1-Wire 1"
+		(property "Value" "DS1820"
 			(at 33.528 126.492 0)
 			(show_name no)

Commit message: kicad: drop Pi Zero holes next to the header, J19 value from board to schematic
H7/H8 and their standoff keep-outs removed: the box header no longer
collides with them (last DRC errors gone), the Zero's header side is held by
the plug connection and its outer side by H5/H6. J19 value "1-wire\nDS1820"
taken over from the board. README/BOM: 2 standoffs instead of 4.

Co-Authored-By: Claude Opus 5.5 <noreply@anthropic.com>
Parts:
- J19: value DS1820 -> 1-wire DS1820
Changed lines of the file:
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@@
 			)
 		)
-		(property "Value" "DS1820"
+		(property "Value" "1-wire\nDS1820"
 			(at 33.528 126.492 0)
 			(show_name no)
