File: kicad/io.kicad_sch (KiCad schematic)
At the start: 23 parts, among them J15 GPIO 5, J16 GPIO 6, J17 GPIO 20, J18 GPIO 21, J19 1-wire DS1820, J22 I2C 1, J23 I2C 2, J24 Display

Commit message: kicad: schematic re-save (library symbol refresh, BOM field setup)
Parts:
- D22, D23, D24, D25, D26: KiLib_Generator (none) -> package/gullwing
- J15, J16, J17, J18, J19: KiLib_Generator (none) -> terminal_block/Phoenix
- J22, J23, J24, JP3: KiLib_Generator (none) -> connector/pin_header_socket
- R36, R37, R38, R39, R40, R41, R42, R43, R44: KiLib_Generator (none) -> SMD_2terminal_chip_molded
